File: ErgoDOX pcb/ErgoDOX.sch (KiCad schematic (older format))
At the start: 97 parts, among them J1 USB, J2 3.5mm, J3 JMP, J4 JMP, SW0:10 SW0:3, SW0:11 SW0:2, SW0:12 SW0:1, SW0:7 SW0:6, SW0:8 SW0:5, SW0:9 SW0:4, SW1:10 SW1:3, SW1:11 SW1:2, SW1:12 SW1:1, SW1:13 SW1:0, SW1:9 SW1:4, SW2:10 SW2:3, SW2:11 SW2:2, SW2:12 SW2:1, SW2:13 SW2:0, SW2:7 SW2:6, SW2:8 SW2:5, SW2:9 SW2:4, SW3:10 SW3:3, SW3:11 SW3:2, SW3:12 SW3:1, SW3:13 SW3:0, SW3:8 SW3:5, SW3:9 SW3:4, SW4:10 SW4:3, SW4:11 SW4:2, SW4:12 SW4:1, SW4:13 SW4:0, SW4:7 SW4:6, SW4:8 SW4:5, SW4:9 SW4:4, SW5:10 SW5:3, SW5:11 SW5:2, SW5:12 SW5:1, SW5:13 SW5:0, SW5:7 SW5:6, SW5:8 SW5:5, SW5:9 SW5:4, U1 TEENSY2.0, U2 MCP23018

Commit message: WIP placement.py script, some routing
Parts:
- added D1:10: D1:3, ErgoDOX pcb:D_DO-35_SOD27_P7.62mm_Horizontal, symbol ErgoDOX-rescue:DIODE
- added D1:11: D1:2, ErgoDOX pcb:D_DO-35_SOD27_P7.62mm_Horizontal, symbol ErgoDOX-rescue:DIODE
- added D1:12: D1:1, ErgoDOX pcb:D_DO-35_SOD27_P7.62mm_Horizontal, symbol ErgoDOX-rescue:DIODE
- added D1:13: D1:0, ErgoDOX pcb:D_DO-35_SOD27_P7.62mm_Horizontal, symbol ErgoDOX-rescue:DIODE
- added D1:9: D1:4, ErgoDOX pcb:D_DO-35_SOD27_P7.62mm_Horizontal, symbol ErgoDOX-rescue:DIODE
- D0:10: renamed from D1:4; value D -> D0:3; footprint DIODE -> ErgoDOX pcb:D_DO-35_SOD27_P7.62mm_Horizontal
- D0:11: renamed from D1:5; value D -> D0:2; footprint DIODE -> ErgoDOX pcb:D_DO-35_SOD27_P7.62mm_Horizontal
- D0:12: renamed from D1:6; value D -> D0:1; footprint DIODE -> ErgoDOX pcb:D_DO-35_SOD27_P7.62mm_Horizontal
- D0:7: renamed from D1:1; value D -> D0:6; footprint DIODE -> ErgoDOX pcb:D_DO-35_SOD27_P7.62mm_Horizontal
- D0:8: renamed from D1:2; value D -> D0:5; footprint DIODE -> ErgoDOX pcb:D_DO-35_SOD27_P7.62mm_Horizontal
- D0:9: renamed from D1:3; value D -> D0:4; footprint DIODE -> ErgoDOX pcb:D_DO-35_SOD27_P7.62mm_Horizontal
- D1:7: value D -> D1:6; footprint DIODE -> ErgoDOX pcb:D_DO-35_SOD27_P7.62mm_Horizontal
- D1:8: value D -> D1:5; footprint DIODE -> ErgoDOX pcb:D_DO-35_SOD27_P7.62mm_Horizontal
- D2:10: renamed from D24; value DIODE -> D2:3; footprint Diode_THT:D_DO-35_SOD27_P7.62mm_Horizontal -> ErgoDOX pcb:D_DO-35_SOD27_P7.62mm_Horizontal
- D2:11: renamed from D25; value DIODE -> D2:2; footprint Diode_THT:D_DO-35_SOD27_P7.62mm_Horizontal -> ErgoDOX pcb:D_DO-35_SOD27_P7.62mm_Horizontal
- D2:12: renamed from D26; value DIODE -> D2:1; footprint Diode_THT:D_DO-35_SOD27_P7.62mm_Horizontal -> ErgoDOX pcb:D_DO-35_SOD27_P7.62mm_Horizontal
- D2:13: renamed from D27; value DIODE -> D2:0; footprint Diode_THT:D_DO-35_SOD27_P7.62mm_Horizontal -> ErgoDOX pcb:D_DO-35_SOD27_P7.62mm_Horizontal
- D2:7: renamed from D21; value DIODE -> D2:6; footprint Diode_THT:D_DO-35_SOD27_P7.62mm_Horizontal -> ErgoDOX pcb:D_DO-35_SOD27_P7.62mm_Horizontal
- D2:8: renamed from D22; value DIODE -> D2:5; footprint Diode_THT:D_DO-35_SOD27_P7.62mm_Horizontal -> ErgoDOX pcb:D_DO-35_SOD27_P7.62mm_Horizontal
- D2:9: renamed from D23; value DIODE -> D2:4; footprint Diode_THT:D_DO-35_SOD27_P7.62mm_Horizontal -> ErgoDOX pcb:D_DO-35_SOD27_P7.62mm_Horizontal
- D3:10: renamed from D14; value DIODE -> D3:3; footprint Diode_THT:D_DO-35_SOD27_P7.62mm_Horizontal -> ErgoDOX pcb:D_DO-35_SOD27_P7.62mm_Horizontal
- D3:11: renamed from D16; value DIODE -> D3:2; footprint Diode_THT:D_DO-35_SOD27_P7.62mm_Horizontal -> ErgoDOX pcb:D_DO-35_SOD27_P7.62mm_Horizontal
- D3:12: renamed from D18; value DIODE -> D3:1; footprint Diode_THT:D_DO-35_SOD27_P7.62mm_Horizontal -> ErgoDOX pcb:D_DO-35_SOD27_P7.62mm_Horizontal
- D3:13: renamed from D20; value DIODE -> D3:0; footprint Diode_THT:D_DO-35_SOD27_P7.62mm_Horizontal -> ErgoDOX pcb:D_DO-35_SOD27_P7.62mm_Horizontal
- D3:8: renamed from D10; value DIODE -> D3:5; footprint Diode_THT:D_DO-35_SOD27_P7.62mm_Horizontal -> ErgoDOX pcb:D_DO-35_SOD27_P7.62mm_Horizontal
- D3:9: renamed from D12; value DIODE -> D3:4; footprint Diode_THT:D_DO-35_SOD27_P7.62mm_Horizontal -> ErgoDOX pcb:D_DO-35_SOD27_P7.62mm_Horizontal
- D4:10: renamed from D13; value DIODE -> D4:3; footprint Diode_THT:D_DO-35_SOD27_P7.62mm_Horizontal -> ErgoDOX pcb:D_DO-35_SOD27_P7.62mm_Horizontal
- D4:11: renamed from D15; value DIODE -> D4:2; footprint Diode_THT:D_DO-35_SOD27_P7.62mm_Horizontal -> ErgoDOX pcb:D_DO-35_SOD27_P7.62mm_Horizontal
- D4:12: renamed from D17; value DIODE -> D4:1; footprint Diode_THT:D_DO-35_SOD27_P7.62mm_Horizontal -> ErgoDOX pcb:D_DO-35_SOD27_P7.62mm_Horizontal
- D4:13: renamed from D19; value DIODE -> D4:0; footprint Diode_THT:D_DO-35_SOD27_P7.62mm_Horizontal -> ErgoDOX pcb:D_DO-35_SOD27_P7.62mm_Horizontal
- D4:7: renamed from D8; value DIODE -> D4:6; footprint Diode_THT:D_DO-35_SOD27_P7.62mm_Horizontal -> ErgoDOX pcb:D_DO-35_SOD27_P7.62mm_Horizontal
- D4:8: renamed from D9; value DIODE -> D4:5; footprint Diode_THT:D_DO-35_SOD27_P7.62mm_Horizontal -> ErgoDOX pcb:D_DO-35_SOD27_P7.62mm_Horizontal
- D4:9: renamed from D11; value DIODE -> D4:4; footprint Diode_THT:D_DO-35_SOD27_P7.62mm_Horizontal -> ErgoDOX pcb:D_DO-35_SOD27_P7.62mm_Horizontal
- D5:10: renamed from D4; value DIODE -> D5:3; footprint Diode_THT:D_DO-35_SOD27_P7.62mm_Horizontal -> ErgoDOX pcb:D_DO-35_SOD27_P7.62mm_Horizontal
- D5:11: renamed from D5; value DIODE -> D5:2; footprint Diode_THT:D_DO-35_SOD27_P7.62mm_Horizontal -> ErgoDOX pcb:D_DO-35_SOD27_P7.62mm_Horizontal
- D5:12: renamed from D6; value DIODE -> D5:1; footprint Diode_THT:D_DO-35_SOD27_P7.62mm_Horizontal -> ErgoDOX pcb:D_DO-35_SOD27_P7.62mm_Horizontal
- D5:13: renamed from D7; value DIODE -> D5:0; footprint Diode_THT:D_DO-35_SOD27_P7.62mm_Horizontal -> ErgoDOX pcb:D_DO-35_SOD27_P7.62mm_Horizontal
- D5:7: renamed from D1; value DIODE -> D5:6; footprint Diode_THT:D_DO-35_SOD27_P7.62mm_Horizontal -> ErgoDOX pcb:D_DO-35_SOD27_P7.62mm_Horizontal
- D5:8: renamed from D2; value DIODE -> D5:5; footprint Diode_THT:D_DO-35_SOD27_P7.62mm_Horizontal -> ErgoDOX pcb:D_DO-35_SOD27_P7.62mm_Horizontal
- D5:9: renamed from D3; value DIODE -> D5:4; footprint Diode_THT:D_DO-35_SOD27_P7.62mm_Horizontal -> ErgoDOX pcb:D_DO-35_SOD27_P7.62mm_Horizontal
- SW1:10, SW1:11, SW1:12, SW1:13, SW1:9: symbol ErgoDOX-rescue:SWITCH_DIODE -> ErgoDOX-rescue:SWITCH_PUSH
- renumbered SW_RST1 to RST_SW1
Connections:
- net COL0: now also D1:13.2 (K); no longer SW1:13.4 (K)
- net COL1: now also D1:12.2 (K); no longer SW1:12.4 (K)
- net COL10: now also D1:10.2 (K); no longer SW1:10.4 (K)
- net COL11: now also D1:11.2 (K); no longer SW1:11.4 (K)
- net COL4: now also D1:9.2 (K); no longer SW1:9.4 (K)
- net at SW1:9.2: now also D1:9.1 (A); no longer SW1:9.3 (A)
- net at SW1:10.2: now also D1:10.1 (A); no longer SW1:10.3 (A)
- net at SW1:12.2: now also D1:12.1 (A); no longer SW1:12.3 (A)
- net at SW1:13.2: now also D1:13.1 (A); no longer SW1:13.3 (A)
- net at SW1:11.2: now also D1:11.1 (A); no longer SW1:11.3 (A)
